File: Schaltung/Bogenampel_embedded.kicad_sch (KiCad schematic)
At the start: 35 parts, among them J1 WS2812B Stripe Timer, J10 Display, J2 Conn_01x04_Pin, J3 DC/DC Boost, J4 Jumper: 5V/Ext Voltage, J5 Buzzer, J6 Battery, J9 Power Bank, Q1 IRLZ44N, U1 NRF24L01_Breakout, U2 TXS0108EPW, U3 LM1117DT-3.3

Commit message: Dokumentation aktualisiert und Schaltung Version 2.2
- HARDWARE.md: Pin-Belegungen korrigiert (NRF D9/D8, Buttons D5/D6/D7, Voltage A5, Buzzer D4)
- README.md: Features, Pin-Tabellen und Kommunikation aktualisiert (158 LEDs, 11 Kommandos)
- Sender/README.md: Alle Features als implementiert markiert, State Machine erweitert
- Sender/SETUP.md: Test-Sektion aktualisiert
- CLAUDE.md: Komplett überarbeitet mit aktuellem Projekt-Stand
- Schaltung: Version 2.2 - bereit für Fertigung
- Test-Dateien entfernt (TestEmpfaenger, TestSender)

🤖 Generated with [Claude Code](https://claude.com/claude-code)

Co-Authored-By: Claude Sonnet 4.5 <noreply@anthropic.com>
Parts:
- added C11, C12: 18 pF, Capacitor_SMD:C_1206_3216Metric, symbol Device:C_Small
- added C13: 100nF, Capacitor_SMD:C_1206_3216Metric, symbol Device:C_Small
- added C14, C15: 10µF, Capacitor_SMD:C_1206_3216Metric, symbol Device:C_Small
- added C16: 100 nF, Capacitor_SMD:C_1206_3216Metric, symbol Device:C_Small
- added J11: Battery, Connector_JST:JST_XH_B2B-XH-A_1x02_P2.50mm_Vertical, symbol Connector:Conn_01x02_Pin
- added J12: RESET, Connector_JST:JST_XH_B2B-XH-A_1x02_P2.50mm_Vertical, symbol Connector:Conn_01x02_Pin
- added J13: PROG, symbol Connector:Conn_01x06_Pin
- added R10: 10kΩ, Resistor_SMD:R_1206_3216Metric, symbol Device:R_Small
- added U4: ATmega328P-A, Package_QFP:TQFP-32_7x7mm_P0.8mm, symbol MCU_Microchip_ATmega:ATmega328P-A
- added U5: LM1117DT-5.0, Package_TO_SOT_SMD:TO-252-3_TabPin2, symbol Regulator_Linear:LM1117DT-3.3
- added Y1: Crystal, symbol Device:Crystal
Connections:
- net +5V: now also C13.1, C14.1, J13.3 (Pin_3), R10.2, U4.18 (AVCC), U4.20 (AREF), U4.4 (VCC), U4.6 (VCC), U5.2 (VO)
- net +BATT: no longer A1.30 (VIN), R7.2
- net GND: now also C11.1, C12.1, C13.2, C14.2, C15.2, J11.1 (Pin_1), J12.1 (Pin_1), J13.1 (Pin_1), U4.21 (GND), U4.3 (GND), U4.5 (GND), U5.1 (GND)
- new net: C16.1, J12.2 (Pin_2), R10.1, U4.29 (~{RESET}/PC6)
- new net: C16.2, J13.6 (Pin_6)
- new net: C11.2, U4.7 (XTAL1/PB6), Y1.2
- new net: C15.1, J11.2 (Pin_2), R7.2, U5.3 (VI)
- new net: J13.4 (Pin_4), U4.30 (PD0)
- new net: J13.5 (Pin_5), U4.31 (PD1)
- new net: C12.2, U4.8 (XTAL2/PB7), Y1.1
Other:
- note added: "Spannungsversorgung Batterie"
- note removed: "Batterie Monitor"
- moved on the sheet: RV1
