File: Schaltung/Bogenampel.kicad_sch (KiCad schematic)
At the start: 35 parts, among them J1 WS2812B Stripe Timer, J10 Display, J2 Conn_01x04_Pin, J3 DC/DC Boost, J4 Jumper: 5V/Ext Voltage, J5 Buzzer, J6 Battery, J9 Power Bank, Q1 IRLZ44N, U1 NRF24L01_Breakout, U2 TXS0108EPW, U3 LM1117DT-3.3

Commit message: Bug: A6 & A7 durch A2 & A3 ersetzt für Digital Output
Co-Authored-By: Claude Opus 4.5 <noreply@anthropic.com>
Connections:
- net DSPL_CS_5V: now also A1.21 (A2); no longer A1.25 (A6)
- net DSPL_RES_5V: now also A1.22 (A3); no longer A1.26 (A7)
Changed lines of the file:
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@@
+	(wire
+		(pts
+			(xy 121.92 111.76) (xy 143.51 111.76)
+		)
+		(stroke
+			(width 0)
+			(type default)
+		)
+	)
 	(wire
 		(pts
@@
 	(wire
 		(pts
+			(xy 121.92 114.3) (xy 139.7 114.3)
+		)
+		(stroke
+			(width 0)
+			(type default)
+		)
+	)
+	(wire
+		(pts
 			(xy 82.55 104.14) (xy 96.52 104.14)
 		)
@@
 	(wire
 		(pts
+			(xy 139.7 114.3) (xy 139.7 124.46)
+		)
+		(stroke
+			(width 0)
+			(type default)
+		)
+	)
+	(wire
+		(pts
 			(xy 156.21 40.64) (xy 128.27 40.64)
 		)
@@
 	(wire
 		(pts
-			(xy 121.92 124.46) (xy 208.28 124.46)
-		)
-		(stroke
-			(width 0)
-			(type default)
-		)
-	)
-	(wire
-		(pts
 			(xy 87.63 58.42) (xy 87.63 101.6)
 		)
@@
 	(wire
 		(pts
+			(xy 143.51 111.76) (xy 143.51 121.92)
+		)
+		(stroke
+			(width 0)
+			(type default)
+		)
+	)
+	(wire
+		(pts
 			(xy 52.07 26.67) (xy 52.07 29.21)
 		)
@@
 	(wire
 		(pts
+			(xy 143.51 121.92) (xy 208.28 121.92)
+		)
+		(stroke
+			(width 0)
+			(type default)
+		)
+	)
+	(wire
+		(pts
+			(xy 139.7 124.46) (xy 208.28 124.46)
+		)
+		(stroke
+			(width 0)
+			(type default)
+		)
+	)
+	(wire
+		(pts
 			(xy 237.49 119.38) (xy 237.49 110.49)
 		)
@@
 		(pts
 			(xy 135.89 57.15) (xy 135.89 109.22)
-		)
-		(stroke
-			(width 0)
-			(type default)
-		)
-	)
-	(wire
-		(pts
-			(xy 121.92 121.92) (xy 208.28 121.92)
 		)
 		(stroke
@@
 	)
 	(label "DSPL_CS_5V"
-		(at 123.19 121.92 0)
+		(at 123.19 111.76 0)
 		(effects
 			(font
@@
 	)
 	(label "DSPL_RES_5V"
-		(at 123.19 124.46 0)
-		(effects
-			(font
+		(at 123.19 114.3 0)
+		(effects
+			(font
