File: Schaltung_v3/BogenampelV3/BogenampelV3.kicad_sch (KiCad schematic)
At the start: 48 parts, among them IC1 TPS62742DSSR, J1 Conn_01x24_Pin, Q1 IRLML9301, Q2 IRLML6346, Q3 Si1308EDL, SW1 SW_Push, SW2 SW_Push, U1 XIAO ESP32C3

Commit message: Universalfernbedienung V3
Parts:
- removed R14: 10k, Resistor_SMD:R_1206_3216Metric, symbol Device:R
- removed U1: XIAO ESP32C3, 0liver:xiao_esp32c3_ohneBat, symbol 0liver:XIAO ESP32C3
- added C15, C17: 4,7µF, Capacitor_SMD:C_0805_2012Metric, symbol Device:C
- added C16, C19: 100nF, Capacitor_SMD:C_0603_1608Metric, symbol Device:C
- added C18: 10µF, Capacitor_SMD:C_0805_2012Metric, symbol Device:C
- added C20: 1µF, Capacitor_SMD:C_0805_2012Metric, symbol Device:C
- added FB1: 220, Resistor_SMD:R_0805_2012Metric, symbol Device:FerriteBead
- added IC2: ESP32-S3-WROOM-1U-N16R8, SamacSys_Parts:ESP32S3WROOM1UN16R8, symbol SamacSys_Parts:ESP32-S3-WROOM-1U-N16R8
- added IC3: MCP73837T-FCI_UN, SamacSys_Parts:SOP50P490X110-10N, symbol SamacSys_Parts:MCP73837T-FCI_UN
- added J2: UJ20-C-H-G-MSMT-4B-P16-TR, SamacSys_Parts:UJ20CHGMSMT4BP16TR, symbol SamacSys_Parts:UJ20-C-H-G-MSMT-4B-P16-TR
- added J3: NTC, Connector_PinHeader_2.54mm:PinHeader_1x02_P2.54mm_Vertical, symbol PCM_PinHeader_Generic_2.54mm:PinHeader_01x02_2.54mm_Vertical
- added J4: BAT, Connector_PinHeader_2.54mm:PinHeader_1x02_P2.54mm_Vertical, symbol PCM_PinHeader_Generic_2.54mm:PinHeader_01x02_2.54mm_Vertical
- added R15, R16: 5k1, Resistor_SMD:R_1206_3216Metric, symbol Device:R
- added R17, R18, R20: 100k, Resistor_SMD:R_1206_3216Metric, symbol Device:R
- added R19: 2k, Resistor_SMD:R_1206_3216Metric, symbol Device:R
- added R21, R22, R23, R24, R25: 10k, Resistor_SMD:R_1206_3216Metric, symbol Device:R
- added SW3: Enable, Button_Switch_THT:SW_PUSH_6mm_H5mm, symbol Switch:SW_Push
- added SW4: Boot, Button_Switch_THT:SW_PUSH_6mm_H5mm, symbol Switch:SW_Push
- added U2: USBLC6-2SC6, Package_TO_SOT_SMD:SOT-23-6, symbol Power_Protection:USBLC6-2SC6
- TP1, TP2, TP3, TP5, TP6: footprint TestPoint:TestPoint_THTPad_1.5x1.5mm_Drill0.7mm -> TestPoint:TestPoint_Pad_D1.5mm
- TP4: footprint TestPoint:TestPoint_THTPad_1.5x1.5mm_Drill0.7mm -> TestPoint:TestPoint_Pad_1.5x1.5mm
Connections:
- net +3V3: now also C18.2, C19.2, IC2.2 (3V3), R21.1, R22.1, R23.1
- net +BATT: now also C17.1, IC3.10 (VBAT), J4.2 (Pin_2)
- net BUSY: now also IC2.31 (IO38)
- net CS_D: now also IC2.23 (IO21)
- net DC: now also IC2.24 (IO47)
- net GND: now also C15.2, C16.2, C17.2, C18.1, C19.1, C20.2, IC2.1 (GND_1), IC2.40 (GND_2), IC2.41 (GND_3), IC2.42 (GND_4), IC2.43 (GND_5), IC2.44 (GND_6), IC2.45 (GND_7), IC2.46 (GND_8), IC2.47 (GND_9), IC2.48 (GND_10), IC2.49 (GND_11), IC3.5 (VSS), J2.A1 (GND_1), J2.B1 (GND_2), J2.MH1 (MH_1), J2.MH2 (MH_2), J2.MH3 (MH_3), J2.MH4 (MH_4), J3.1 (Pin_1), J4.1 (Pin_1), R15.2, R16.2, R18.1, R19.2, R20.2, R24.1, R25.1, SW3.1, SW4.1, U2.2 (GND)
- net RES: now also IC2.25 (IO48)
- net ADC_BATT_SENS renamed ADC_BAT
- net ADC_BAT: now also IC2.18 (IO10)
- net GPIO_BTN1 renamed BTN1
- net BTN1: now also IC2.8 (IO15)
- net GPIO_BTN2 renamed BTN2
- net BTN2: now also IC2.17 (IO9)
- net GPIO_LATCH renamed LATCH
- net LATCH: now also IC2.9 (IO16)
- net GPIO_LOAD renamed LOAD
- net LOAD: now also IC2.7 (IO7)
- net NC: no longer names the net of J1.1 (Pin_1)
- net NC: no longer J1.4 (Pin_4)
- net SCL renamed CLK
- net CLK: now also IC2.22 (IO14)
- net SDA renamed MOSI
- net MOSI: now also IC2.21 (IO13)
- net TSCL: no longer names the net of J1.6 (Pin_6)
- net TSDA: no longer names the net of J1.7 (Pin_7)
- net VPP: no longer names the net of J1.19 (Pin_19)
- new net: IC3.6 (PROG1), R19.1
- new net: IC3.9 (THERM), J3.2 (Pin_2)
- new net: FB1.2, J2.A4 (VBUS_1), J2.B4 (VBUS_2)
- new net: J2.A5 (CC1), R15.1
- new net: J2.B5 (CC2), R16.1
- new net: IC2.15 (IO3), R23.2
- new net: IC2.16 (IO46), R25.2
- new net: IC2.26 (IO45), R24.2
- new net: IC2.27 (IO0), R22.2, SW4.2
- new net: C20.1, IC2.3 (EN), R21.2, SW3.2
- new net C_PG: IC2.10 (IO17), IC3.8 (~{PG_(}TE))
- new net C_PRG: IC2.11 (IO18), IC3.7 (PROG2), R20.1
- new net C_ST1: IC2.19 (IO11), IC3.3 (STAT1)
- new net C_ST2: IC2.20 (IO12), IC3.4 (STAT2)
- new net DN: J2.A7 (DN1), J2.B7 (DN2), U2.1 (I/O1)
- new net DP: J2.A6 (DP1), J2.B6 (DP2), U2.3 (I/O2)
- new net USB_CON: IC2.12 (IO8), R17.1, R18.2
- new net USB_D+: IC2.14 (IO20), U2.4 (I/O2)
- new net USB_D-: IC2.13 (IO19), U2.6 (I/O1)
- new net VCC: C15.1, C16.1, FB1.1, IC3.2 (VUSB), R17.2, U2.5 (VBUS)
- no-connect marks 0 -> 23
Other:
- note added: "Battery Voltage Sensor (stromlos wenn aus)"
- note added: "DCDC BAT - 3V3"
- note added: "Laderregler"
- note added: "One-Button Power on"
- note added: "USB Connector"
- note added: "Waveshare 1.5'' e-Paper V2"
- note added: "µController"
- note removed: "Waveshare 1.5inch e-Paper V2"
- title: (none) -> Universal-Fernbedienung ESP32
- moved on the sheet: C1, C10, C11, C12, C13, C14, C2, C3, C4, C5, C6, C7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
