File: Schaltung_v3/BogenampelV3/BogenampelV3.kicad_sch (KiCad schematic)
At the start: 72 parts, among them IC1 TPS62742DSSR, IC2 ESP32-S3-WROOM-1U-N16R8, IC3 MCP73837T-FCI_UN, J1 Conn_01x24_Pin, J2 UJ20-C-H-G-MSMT-4B-P16-TR, J3 NTC, J4 BAT, Q1 IRLML9301, Q2 IRLML6346, Q3 Si1308EDL, SW1 SW_Push, SW2 SW_Push, SW3 Enable, SW4 Boot, U2 USBLC6-2SC6

Commit message: V3-Firmware: OTA, zentrales PlatformIO, .cpp-Umbenennung, Lüfter-Fix
- EmpfaengerV3 + SenderV3: .ino → .cpp (kein Konverter-Schritt mehr)
- OTA via ArduinoOTA: SoftAP-Fallback + STA-Modus (DHCP, wifi_credentials.h)
- Zentrales platformio.ini im Repo-Root (extends, build_src_filter)
- FanManager: Gate-Duty invertiert (Q2 Open-Drain, Poti-Richtung korrigiert)
- Lochrasterskizze: POTI_GND-Trennschnitt und Lüfter-Netz-Kurzschluss behoben
- KiCad: Gerber-Export, STEP-Modelle, aktualisierter Empfänger-Schaltplan
- wifi_credentials.h.example als Vorlage (echte Datei gitignored)

Co-Authored-By: Claude Sonnet 4.6 <noreply@anthropic.com>
Parts:
- R7: value 47k -> 240k
Changed lines of the file:
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@@
 			)
 		)
-		(property "Value" "47k"
+		(property "Value" "240k"
 			(at 138.43 81.2799 0)
 			(show_name no)
