File: Schaltung-Empfaenger/Empfaenger.kicad_sch (KiCad schematic)
At the start: 44 parts, among them J1 Conn_01x06 USB, J2 Poti 47k, J3 Poti 47k, J4 Poti 47k, J5 BTN, J6 Fan, J7 LED Stripe, J8 Piezo Transducter 12V, Q1 IRLML9301, Q2 2N7002, Q3 BC337, U1 L7805, U2 CH224K, U3 XIAO ESP32C3, U4 TSR0.5-2433, U5 74AHCT1G125

Commit message: Empfaenger: PCB fertig geroutet
Layout des Empfaenger-Boards abgeschlossen.

PCB
- Leiterbahnen 100 -> 323 Segmente, Vias 4 -> 10: das Board ist jetzt
  durchgeroutet statt teilverdrahtet
- Zweite Kupferflaeche hinzugekommen (1 -> 2 Zonen)
- Platinenumriss gezeichnet (4 gr_line)
- C11 platziert (44 -> 45 Footprints)

Schaltplan
- C11 (1µF, 1206) und die Versorgung VDD_PD ergaenzt, dazu zwei
  Power-Symbole (#PWR052/053) sowie 2k2 und 470 Ohm
- 14 Widerstaende von 1206 auf 0603 umgestellt

Die Netz-Labels sind unveraendert — der Pin-Contract aus
specs/004-v3-esp32-port/contracts/hardware-pins.md gilt weiter, die
Empfaenger-Firmware ist von dieser Aenderung nicht betroffen.

Co-Authored-By: Claude Opus 5 (1M context) <noreply@anthropic.com>
Parts:
- added C11: 1µF, Capacitor_SMD:C_1206_3216Metric, symbol Device:C
- R10, R11, R12, R13, R14, R2, R3, R4, R5, R6, R7, R8, R9: footprint Resistor_SMD:R_1206_3216Metric -> Resistor_SMD:R_0603_1608Metric
- R15: value 470 -> 2k2; footprint Resistor_SMD:R_1206_3216Metric -> Resistor_SMD:R_0603_1608Metric
Connections:
- net +3V3: no longer C3.1, R1.2, U2.1 (VDD), U2.3 (CFG3)
- net GND: now also C11.2
- new net VDD_PD: C11.1, C3.1, R1.2, U2.1 (VDD), U2.3 (CFG3)
Other:
- moved on the sheet: C3, R6
