File: Schaltung-Empfaenger/Empfaenger.kicad_sch (KiCad schematic)
At the start: 45 parts, among them J1 Conn_01x06 USB, J2 Poti 47k, J3 Poti 47k, J4 Poti 47k, J5 BTN, J6 Fan, J7 LED Stripe, J8 Piezo Transducter 12V, Q1 IRLML9301, Q2 2N7002, Q3 BC337, U1 L7805, U2 CH224K, U3 XIAO ESP32C3, U4 TSR0.5-2433, U5 74AHCT1G125

Commit message: Finale überarbeitung (Druck, Bohrlöcher, TP) vor Fertigung
Parts:
- added TP1: +3V3, TestPoint:TestPoint_Pad_D1.5mm, symbol Connector:TestPoint
- added TP2: VPD, TestPoint:TestPoint_Pad_D1.5mm, symbol Connector:TestPoint
- added TP3: +5V, TestPoint:TestPoint_Pad_D1.5mm, symbol Connector:TestPoint
Connections:
- net +3V3: now also TP1.1
- net +5V: now also TP3.1
- net VDD_PD: now also TP2.1
- net SIG_LED: now reaches U3.11 (D10), U5.2
Other:
- title: (none) -> Bogenampel Empfänger
- moved on the sheet: C1, C11, C2, C3, C4, C5, C6, C7, C8, C9, D2, Q1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
