File: Schaltung-Empfaenger/Empfaenger.kicad_sch (KiCad schematic)
At the start: 48 parts, among them J1 Conn_01x06 USB, J2 Poti 47k, J3 Poti 47k, J4 Poti 47k, J5 BTN, J6 Fan, J7 LED Stripe, J8 Piezo Transducter 12V, Q1 IRLML9301, Q2 2N7002, Q3 BC337, U1 L7805, U2 CH224K, U3 XIAO ESP32C3, U4 TSR0.5-2433, U5 74AHCT1G125

Commit message: Empfaenger-Platine: Bemassungen, MOSFET-Typen und BOM-Export
- PCB: Bemassungen auf User.1 ergaenzt (Bohrabstaende/Platinenmasse)
- Schaltplan: Q1 IRLML9301 -> AO3401A, Q2 2N7002 -> BSS138
- BOM-Export Empfaenger.csv hinzugefuegt (Stand vor der MOSFET-Umbenennung)
- BOM-Spalten (MPN/MFG/Beschreibung) im Projekt konfiguriert

Co-Authored-By: Claude Opus 5 (1M context) <noreply@anthropic.com>
Parts:
- Q1: value IRLML9301 -> AO3401A
- Q2: value 2N7002 -> BSS138
Changed lines of the file:
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@@
 			)
 		)
-		(property "Value" "2N7002"
+		(property "Value" "BSS138"
 			(at 223.52 93.9799 0)
 			(show_name no)
@@
 			)
 		)
-		(property "Value" "IRLML9301"
+		(property "Value" "AO3401A"
 			(at 140.97 43.1799 0)
 			(show_name no)
