File: Schaltung-Empfaenger/Empfaenger.kicad_pcb (KiCad board)
At the start: 2 copper layers, 61 x 43 mm, 45 parts, among them J1 Conn_01x06 USB, J2 Poti 47k, J3 Poti 47k, J4 Poti 47k, J5 BTN, J6 Fan, J7 LED Stripe, J8 Piezo Transducter 12V, Q1 IRLML9301, Q2 2N7002, Q3 BC337, U1 L7805, U2 CH224K, U3 XIAO ESP32C3, U4 TSR0.5-2433, U5 74AHCT1G125

Commit message: Finale überarbeitung (Druck, Bohrlöcher, TP) vor Fertigung
Parts:
- added REF**1: MountingHole_2.2mm_M2, MountingHole:MountingHole_2.2mm_M2, F.Cu at (114.0, 123.0)
- added REF**2: MountingHole_2.2mm_M2, MountingHole:MountingHole_2.2mm_M2, F.Cu at (162.0, 95.0)
- added REF**3: MountingHole_2.2mm_M2, MountingHole:MountingHole_2.2mm_M2, F.Cu at (169.0, 123.0)
- added TP1: +3V3, TestPoint:TestPoint_Pad_D1.5mm, F.Cu at (165.9, 93.7)
- added TP2: VPD, TestPoint:TestPoint_Pad_D1.5mm, F.Cu at (123.7, 117.1)
- added TP3: +5V, TestPoint:TestPoint_Pad_D1.5mm, F.Cu at (159.3, 117.3)
- moved R6 61.2 mm to (164.3, 91.3)
- moved D2 60.1 mm to (142.9, 116.3)
- moved R1 60.1 mm to (128.8, 117.0)
- moved C3 60.1 mm to (123.5, 113.0)
- moved C8 60.1 mm to (143.3, 107.1)
- moved J1 60.1 mm to (136.0, 122.6)
- moved Q1 60.1 mm to (135.9, 115.3)
- moved Q3 60.1 mm to (122.5, 107.6)
- moved R11 60.1 mm to (159.8, 108.9)
- moved R14 60.1 mm to (159.1, 111.7)
- moved R15 60.1 mm to (136.0, 110.2)
- moved R2 60.1 mm to (128.5, 105.3)
- moved R4 60.1 mm to (121.7, 88.3)
- moved R7 60.1 mm to (132.6, 105.3)
- moved R9 60.1 mm to (153.1, 91.4)
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Connections:
- net /<NO NET> renamed /SIG_LED
Routing:
- net +3V3: track 123.1 -> 128.4 mm
- net VDD_PD: track 11.7 -> 15.4 mm
- net +5V: track 13.4 -> 15.6 mm
- net GND: track 240.2 -> 241.7 mm, vias 0 -> 6
- added copper zone on B.Cu, net GND
- added copper zone on F.Cu, net GND
Other:
- board text added: "Bogenampel V3 08/2026"
